Commit message: fixed the rviz model, still need to cleanout turtlebot related model info, but seems to work with romipi_fake

File: romipi_description/urdf/romipi.urdf.xacro (robot description, xacro)
@@ -7,11 +7,11 @@
     <parent link="base_footprint"/>
     <child link="base_link"/>
-    <origin xyz="0.0 0.0 0.010" rpy="0 0 0"/>
+    <origin xyz="0.0 0.0 0.00" rpy="0 0 0"/>
   </joint>
   <link name="base_link">
     <visual>
-      <origin xyz="-0.032 0 0.0" rpy="0 0 0"/>
+      <origin xyz="0.0 0.0 0.0" rpy="0 0 0"/>
       <geometry>
-        <mesh filename="package://romipi_description/meshes/bases/burger_base.stl" scale="0.001 0.001 0.001"/>
+        <mesh filename="package://romipi_description/meshes/bases/romi_base.stl" scale="1 1 1"/>
       </geometry>
       <material name="light_black"/>
@@ -34,12 +34,12 @@
     <parent link="base_link"/>
     <child link="wheel_left_link"/>
-    <origin xyz="0.0 0.08 0.023" rpy="-1.57 0 0"/>
-    <axis xyz="0 0 1"/>
+    <origin xyz="0.0 0.07 0.0345" rpy="0 0 0"/>
+    <axis xyz="0 1 0"/>
   </joint>
   <link name="wheel_left_link">
     <visual>
-      <origin xyz="0 0 0" rpy="1.57 0 0"/>
+      <origin xyz="0 0.0 0.0" rpy="3.14 0 0"/>
       <geometry>
-        <mesh filename="package://romipi_description/meshes/wheels/left_tire.stl" scale="0.001 0.001 0.001"/>
+        <mesh filename="package://romipi_description/meshes/wheels/romi-left-wheel.stl" scale="1 1 1"/>
       </geometry>
       <material name="dark"/>
@@ -48,5 +48,5 @@
       <origin xyz="0 0 0" rpy="0 0 0"/>
       <geometry>
-        <cylinder length="0.018" radius="0.033"/>
+        <cylinder length="0.018" radius="0.0345"/>
       </geometry>
     </collision>
@@ -62,12 +62,12 @@
     <parent link="base_link"/>
     <child link="wheel_right_link"/>
-    <origin xyz="0.0 -0.080 0.023" rpy="-1.57 0 0"/>
-    <axis xyz="0 0 1"/>
+    <origin xyz="0.0 -0.07 0.0345" rpy="0 0 0"/>
+    <axis xyz="0 1 0"/>
   </joint>
   <link name="wheel_right_link">
     <visual>
-      <origin xyz="0 0 0" rpy="1.57 0 0"/>
+      <origin xyz="0 0 0" rpy="0 0 0"/>
       <geometry>
-        <mesh filename="package://romipi_description/meshes/wheels/right_tire.stl" scale="0.001 0.001 0.001"/>
+        <mesh filename="package://romipi_description/meshes/wheels/romi-right-wheel.stl" scale="1 1 1"/>
       </geometry>
       <material name="dark"/>

Commit message: added the back castor

File: romipi_description/urdf/romipi.urdf.xacro (robot description, xacro)
@@ -11,5 +11,5 @@
   <link name="base_link">
     <visual>
-      <origin xyz="0.0 0.0 0.0" rpy="0 0 0"/>
+      <origin xyz="0.0 0.0 0.0" rpy="0 0 3.14"/>
       <geometry>
         <mesh filename="package://romipi_description/meshes/bases/romi_base.stl" scale="1 1 1"/>
@@ -18,7 +18,7 @@
     </visual>
     <collision>
-      <origin xyz="-0.032 0 0.070" rpy="0 0 0"/>
+      <origin xyz="0.0 0.0 0.0315" rpy="0 0 0"/>
       <geometry>
-        <box size="0.140 0.140 0.143"/>
+        <box size="0.1635 0.145 0.063"/>
       </geometry>
     </collision>
@@ -46,5 +46,5 @@
     </visual>
     <collision>
-      <origin xyz="0 0 0" rpy="0 0 0"/>
+      <origin xyz="0 0 0" rpy="1.57 0 0"/>
       <geometry>
         <cylinder length="0.018" radius="0.0345"/>
@@ -74,5 +74,5 @@
     </visual>
     <collision>
-      <origin xyz="0 0 0" rpy="0 0 0"/>
+      <origin xyz="0 0 0" rpy="1.57 0 0"/>
       <geometry>
         <cylinder length="0.018" radius="0.033"/>
@@ -90,11 +90,18 @@
     <parent link="base_link"/>
     <child link="caster_back_link"/>
-    <origin xyz="-0.081 0 -0.004" rpy="-1.57 0 0"/>
+    <origin xyz="-0.0441 0 0.0" rpy="0 0 0"/>
   </joint>
   <link name="caster_back_link">
+    <visual>
+      <origin xyz="0 0.0 0.0" rpy="0 0 0"/>
+      <geometry>
+        <mesh filename="package://romipi_description/meshes/wheels/romi-back-castor.stl" scale="1 1 1"/>
+      </geometry>
+      <material name="dark"/>
+    </visual>
     <collision>
-      <origin xyz="0 0.001 0" rpy="0 0 0"/>
+      <origin xyz="0 0.0 0.005" rpy="0 0 0"/>
       <geometry>
-        <box size="0.030 0.009 0.020"/>
+        <box size="0.030 0.02 0.01"/>
       </geometry>
     </collision>
@@ -113,30 +120,3 @@
   </joint>
   <link name="imu_link"/>
-  <joint name="scan_joint" type="fixed">
-    <parent link="base_link"/>
-    <child link="base_scan"/>
-    <origin xyz="-0.032 0 0.172" rpy="0 0 0"/>
-  </joint>
-  <link name="base_scan">
-    <visual>
-      <origin xyz="0 0 0.0" rpy="0 0 0"/>
-      <geometry>
-        <mesh filename="package://romipi_description/meshes/sensors/lds.stl" scale="0.001 0.001 0.001"/>
-      </geometry>
-      <material name="dark"/>
-    </visual>
-    <collision>
-      <origin xyz="0.015 0 -0.0065" rpy="0 0 0"/>
-      <geometry>
-        <cylinder length="0.0315" radius="0.055"/>
-      </geometry>
-    </collision>
-    <inertial>
-      <mass value="0.114" />
-      <origin xyz="0 0 0" />
-      <inertia ixx="0.001" ixy="0.0" ixz="0.0"
-               iyy="0.001" iyz="0.0"
-               izz="0.001" />
-    </inertial>
-  </link>
 </robot>

Commit message: gazebo empty world simulation works and robot can do a little dance

File: romipi_description/urdf/romipi.urdf.xacro (robot description, xacro)
@@ -20,5 +20,5 @@
       <origin xyz="0.0 0.0 0.0315" rpy="0 0 0"/>
       <geometry>
-        <box size="0.1635 0.145 0.063"/>
+        <box size="0.1635 0.145 0.05"/>
       </geometry>
     </collision>

Commit message: Cleaning up urdf description file- romi.urdf.xacro

File: romipi_description/urdf/romipi.urdf.xacro (robot description, xacro)
@@ -3,4 +3,15 @@
   <xacro:include filename="$(find romipi_description)/urdf/common_properties.xacro"/>
   <xacro:include filename="$(find romipi_description)/urdf/romipi.gazebo.xacro"/>
+  <xacro:property name="base_link_mass" value="8.2573504e-01" />
+  <xacro:property name="base_link_colision_l" value="0.1635" />
+  <xacro:property name="base_link_colision_w" value="0.145" />
+  <xacro:property name="base_link_colision_h" value="0.05" />
+  <xacro:property name="wheel_mass" value="2.8498940e-02" />
+  <xacro:property name="wheel_width" value="0.018" />
+  <xacro:property name="wheel_radius" value="0.0345" />
+  <xacro:property name="caster_mass" value="0.0005" />
+  <xacro:property name="caster_colision_l" value="0.01" />
+  <xacro:property name="caster_colision_w" value="0.01" />
+  <xacro:property name="caster_colision_h" value="0.01" />
   <link name="base_footprint"/>
   <joint name="base_joint" type="fixed">
@@ -20,21 +31,18 @@
       <origin xyz="0.0 0.0 0.0315" rpy="0 0 0"/>
       <geometry>
-        <box size="0.1635 0.145 0.05"/>
+        <box size="${base_link_colision_l} ${base_link_colision_w} ${base_link_colision_h}"/>
       </geometry>
     </collision>
     <inertial>
-      <origin xyz="0 0 0.0315" rpy="0 0 0"/>
-      <mass value="8.2573504e-01"/>
+      <origin xyz="0 0 0.0315" rpy="0 0 ${pi/2}"/>
+      <mass value="${base_link_mass}" />
       <!-- According to https://en.wikipedia.org/wiki/List_of_moments_of_inertia#List_of_3D_inertia_tensors
-      We want Ixx = (1/12) * m * (h^2 + l^2) = 0.068811253 * (0.05^2 + 0.1635^2) = 0.002011508 = 2.011508e-03
-              Iyy = (1/12) * m * (w^2 + l^2) = 0.068811253 * (0.145^2 + 0.1635^2) = 0.003286236 = 3.286236e-03
-              Izz = (1/12) * m * (w^2 + h^2) = 0.068811253 * (0.145^2 + 0.05^2) = 0.001618785 = 1.618785e-03
+      We want Ixx = (1/12) * m * (l^2 + h^2) = 0.068811253 * (0.05^2 + 0.1635^2) = 0.002011508 = 2.011508e-03
+              Iyy = (1/12) * m * (w^2 + h^2) = 0.068811253 * (0.145^2 + 0.1635^2) = 0.003286236 = 3.286236e-03
+              Izz = (1/12) * m * (w^2 + l^2) = 0.068811253 * (0.145^2 + 0.05^2) = 0.001618785 = 1.618785e-03
               -->
-      <!--inertia ixx="2.2124416e-03" ixy="-1.2294101e-05" ixz="3.4938785e-05"
-               iyy="2.1193702e-03" iyz="-5.0120904e-06"
-               izz="2.0064271e-03" /-->
-      <inertia ixx="2.011508e-03" ixy="0" ixz="0"
-               iyy="3.286236e-03" iyz="0"
-               izz="1.618785e-03" />
+      <inertia ixx="${(1/12) * base_link_mass * (base_link_colision_l**2 + base_link_colision_h**2)}" ixy="0" ixz="0"
+               iyy="${(1/12) * base_link_mass * (base_link_colision_w**2 + base_link_colision_h**2)}" iyz="0"
+               izz="${(1/12) * base_link_mass * (base_link_colision_w**2 + base_link_colision_l**2)}" />
     </inertial>
   </link>
@@ -42,5 +50,5 @@
     <parent link="base_link"/>
     <child link="wheel_left_link"/>
-    <origin xyz="0.0 0.07 0.0345" rpy="0 0 0"/>
+    <origin xyz="0.0 0.07 ${wheel_radius}" rpy="0 0 0"/>
     <axis xyz="0 1 0"/>
   </joint>
@@ -56,6 +64,5 @@
       <origin xyz="0 0 0" rpy="1.57 0 0"/>
       <geometry>
-        <!--cylinder length="0.018" radius="0.0345"/-->
-        <cylinder length="0.018" radius="0.0345"/>
+        <cylinder length="${wheel_width}" radius="${wheel_radius}"/>
       </geometry>
     </collision>
@@ -63,8 +70,7 @@
       <origin xyz="0 0 0" rpy="1.57 0 0"/>
       <geometry>
-        <!--cylinder length="0.018" radius="0.0345"/-->
-        <cylinder length="0.018" radius="0.0345"/>
+        <cylinder length="${wheel_width}" radius="${wheel_radius}"/>
       </geometry>
-      <mass value="2.8498940e-02" />
+      <mass value="${wheel_mass}" />
       <!-- According to https://en.wikipedia.org/wiki/List_of_moments_of_inertia#List_of_3D_inertia_tensors
       We want Ixx = (1/12) * m * (3*r^2 + h^2) = 0.002374912 * (3 * 0.0345^2 + 0.018^2) = 0.00000925 = 9.25e-06
@@ -72,10 +78,7 @@
               Izz = (1/2) * m * r^2 = 0.01424947 * 0.0345^2 = 0.00001696 = 1.696e-05
               -->
-      <!--inertia ixx="1.1175580e-05" ixy="-4.2369783e-11" ixz="-5.9381719e-09"
-               iyy="1.1192413e-05" iyz="-1.4400107e-11"
-               izz="2.0712558e-05" /-->
-      <inertia ixx="9.25e-06" ixy="0" ixz="0"
-               iyy="9.25e-06" iyz="0"
-               izz="1.696e-05" />
+      <inertia ixx="${(1/12) * wheel_mass * (3 * wheel_radius**2 + wheel_width**2)}" ixy="0" ixz="0"
+               iyy="${(1/12) * wheel_mass * (3 * wheel_radius**2 + wheel_width**2)}" iyz="0"
+               izz="${(1/2) * wheel_mass * wheel_radius**2}" />
       </inertial>
   </link>
@@ -83,5 +86,5 @@
     <parent link="base_link"/>
     <child link="wheel_right_link"/>
-    <origin xyz="0.0 -0.07 0.0345" rpy="0 0 0"/>
+    <origin xyz="0.0 -0.07 ${wheel_radius}" rpy="0 0 0"/>
     <axis xyz="0 1 0"/>
   </joint>
@@ -97,11 +100,10 @@
       <origin xyz="0 0 0" rpy="1.57 0 0"/>
       <geometry>
-        <!--cylinder length="0.018" radius="0.033"/-->
-        <cylinder length="0.018" radius="0.0345"/>
+        <cylinder length="${wheel_width}" radius="${wheel_radius}"/>
       </geometry>
     </collision>
     <inertial>
       <origin xyz="0 0 0" rpy="1.57 0 0"/>
-      <mass value="2.8498940e-02" />
+      <mass value="${wheel_mass}" />
       <!-- According to https://en.wikipedia.org/wiki/List_of_moments_of_inertia#List_of_3D_inertia_tensors
       We want Ixx = (1/12) * m * (3*r^2 + h^2) = 0.002374912 * (3 * 0.0345^2 + 0.018^2) = 0.00000925 = 9.25e-06
@@ -109,10 +111,7 @@
               Izz = (1/2) * m * r^2 = 0.01424947 * 0.0345^2 = 0.00001696 = 1.696e-05
               -->
-      <!--inertia ixx="1.1175580e-05" ixy="-4.2369783e-11" ixz="-5.9381719e-09"
-               iyy="1.1192413e-05" iyz="-1.4400107e-11"
-               izz="2.0712558e-05" /-->
-      <inertia ixx="9.25e-06" ixy="0" ixz="0"
-               iyy="9.25e-06" iyz="0"
-               izz="1.696e-05" />
+      <inertia ixx="${(1/12) * wheel_mass * (3 * wheel_radius**2 + wheel_width**2)}" ixy="0" ixz="0"
+               iyy="${(1/12) * wheel_mass * (3 * wheel_radius**2 + wheel_width**2)}" iyz="0"
+               izz="${(1/2) * wheel_mass * wheel_radius**2}" />
       </inertial>
   </link>
@@ -133,10 +132,10 @@
       <origin xyz="0.0 -0.045 0.005" rpy="0 0 0"/>
       <geometry>
-        <box size="0.01 0.01 0.01"/>
+        <box size="${caster_colision_l} ${caster_colision_w} ${caster_colision_h}"/>
       </geometry>
     </collision>
     <inertial>
       <origin xyz="0 0 0" />
-      <mass value="0.0005" />
+      <mass value="${caster_mass}" />
       <!-- According to https://en.wikipedia.org/wiki/List_of_moments_of_inertia#List_of_3D_inertia_tensors
       We want Ixx = (1/12) * m * (h^2 + l^2) = 0.000041667 * (0.01^2 + 0.01^2) = 0.000000008 = 8e-09
@@ -144,10 +143,7 @@
               Izz = (1/12) * m * (w^2 + h^2) = 0.000041667 * (0.01^2 + 0.01^2) = 0.000000008 = 8e-09
               -->
-      <!--inertia ixx="0.001" ixy="0.0" ixz="0.0"
-               iyy="0.001" iyz="0.0"
-               izz="0.001" /-->
-      <inertia ixx="8e-09" ixy="0" ixz="0"
-               iyy="8e-09" iyz="0"
-               izz="8e-09" />
+      <inertia ixx="${(1/12) * caster_mass * (caster_colision_l**2 + caster_colision_h**2)}" ixy="0" ixz="0"
+               iyy="${(1/12) * caster_mass * (caster_colision_w**2 + caster_colision_h**2)}" iyz="0"
+               izz="${(1/12) * caster_mass * (caster_colision_w**2 + caster_colision_l**2)}" />
     </inertial>
   </link>
